Commit message: Update training pipeline, eval scripts, and docs
Add .gitignore to exclude large training runs/logs/cache.
Add eval scripts (stage1-3, hover, grasp physics tests),
training shell scripts, grasp object asset, and thesis/IROS docs.
Update env, controller, reward, and PPO config for multi-stage training.

Co-Authored-By: Claude Opus 4.6 (1M context) <noreply@anthropic.com>

File: gripper_drone_v5.urdf (robot description, URDF)
Before this commit: robot gripper_drone, 15 links, 14 joints
Links:
- link plate_left: mass 0.055000 -> 0.060000; geometry collision box size=0.012000 0.025000 0.110000; collision box size=0.012000 0.025000 0.110000
- link plate_right: mass 0.055000 -> 0.060000; geometry collision box size=0.012000 0.025000 0.110000; collision box size=0.012000 0.025000 0.110000
